File: transmitter.sch (EAGLE design)
At the start: 20 parts, among them U1 TP4056, U2 XC6206

Commit message: Added initial schematic of transmiter
Parts:
- removed PV_PANEL: JST-2.5MM-1X2, Custom_Parts:JST-2.5MM-1X2
- removed U$1: SX1308, Custom_Parts:SX1308
- added C10, C11, C12, C9: 0.1uF, SparkFun-Capacitors:0.1UF-0603-25V-(+80/-20%)
- added C8: 0.1uF, SparkFun-Capacitors:0.1UF-0603-25V-5%
- added J1: MaxSonar-EZ, SparkFun-Connectors:CONN_07
- added J2: HC-SR04, SparkFun-Connectors:CONN_04
- added PV_PANEL_6V: JST-2.5MM-1X2, Custom_Parts:JST-2.5MM-1X2
- added R6: 10k, SparkFun-Resistors:10KOHM-0603-1/10W-1%
- added U$3: AVR-ISP-6PIN-EDGE, Custom_Parts:AVR-ISP-6PIN-EDGE
- added U3: SX1308, Custom_Parts:SX1308
- added U4: MEGA8-AI, atmel:MEGA8-AI
- added U5: RFM69HCW, Custom_Parts:RFM69HCW
- added Y1: 32.768kHz, SparkFun-Clocks:CRYSTAL-32.768KHZPTH-2X6
- D2: value DIODE-SCHOTTKY -> SS34
Connections:
- new net AVR_RESET: C8.1, R6.1, U$3.RST, U4.PC6(/RESET)
- new net MISO: U$3.MISO, U4.PB4(MISO), U5.MISO
- new net MOSI: U$3.MOSI, U4.PB3(MOSI/OC2), U5.MOSI
- new net N$5: U4.PB6(XTAL1/TOSC1), Y1.1
- new net N$7: U4.PB7(XTAL2/TOSC2), Y1.2
- new net PULSE: J1.2, J2.2, U4.PB0(ICP)
- new net RF_ANT: U5.ANT
- new net RF_RESET: U4.PB1(OC1A), U5.RESET
- new net RX_INT: U4.PD2(INT0), U5.DIO0
- new net SCK: U$3.SCK, U4.PB5(SCK), U5.SCK
- new net SSEL: U4.PB2(SS/OC1B), U5.NSS
- new net TRIGGER: J1.4, J2.3, U4.PD7(AIN1)
- net 3.3V: now also C10.1, C12.1, C9.2, J1.6, R6.2, U$3.VTG, U3.VIN, U4.AVCC, U4.VCC@1, U4.VCC@2, U5.3.3V; no longer U$1.VIN
- net 5V: now also C11.1, J2.4
- net BOOST_EN: now also U3.EN; no longer U$1.EN
- net GND: now also C10.2, C11.2, C12.2, C8.2, C9.1, J1.7, J2.1, PV_PANEL_6V.N, U$3.GND, U3.GND, U4.GND, U4.GND@1, U4.GND@2, U5.GND, U5.GND@10, U5.GND@8; no longer PV_PANEL.N, U$1.GND
- net N$1: now also PV_PANEL_6V.P; no longer PV_PANEL.P
- net N$6: now also U3.SW; no longer U$1.SW
- net N$9: now also U3.FB; no longer U$1.FB
Other:
- moved on the sheet: BATT, C1, C2, C3, C4, C5, C6, C7, D1, D2, L1, R1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
